File: boards/retro-stack-power-clock/retro-stack-power-clock.kicad_pcb (KiCad board)
At the start: 2 copper layers, 99.1 x 99.1 mm, 56 parts, among them J1 BUS_6502, J2 DC_IN, J3 JMP_CLK_SEL, J4 JMP_HLT, SW1 SW_PWR, SW2 SW_MODE, SW3 SW_PULSE, U1 L7805CV, U2 74HC08, U3 74HC32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

Commit message: Rev 0 of the power and clock card ordered.
Parts:
- added REF**: WEEE-Logo_4.2x6mm_SilkScreen, Symbol:WEEE-Logo_4.2x6mm_SilkScreen, B.Cu at (172.1, 43.8)
- added REF**: KiCad-Logo2_6mm_SilkScreen, Symbol:KiCad-Logo2_6mm_SilkScreen, B.Cu at (182.9, 43.2)
- added REF**: Polarity_Center_Positive_6mm_SilkScreen, Symbol:Polarity_Center_Positive_6mm_SilkScreen, B.Cu at (112.4, 57.8)
- moved SW3 153.7 mm to (173.7, 135.2), turned to 180 degrees
- moved NT1 144.0 mm to (189.2, 81.3), turned to 0 degrees
- moved U2 143.0 mm to (163.8, 58.4), turned to 0 degrees
- moved C15 139.7 mm to (170.1, 54.6), turned to 180 degrees
- moved R11 138.5 mm to (190.5, 128.3)
- moved C9 137.0 mm to (184.2, 109.2)
- moved R5 134.2 mm to (161.3, 128.3)
- moved J3 132.1 mm to (181.6, 68.6), turned to 0 degrees
- moved NT2 131.6 mm to (195.6, 115.6), turned to 0 degrees
- moved U7 131.0 mm to (167.6, 106.7), turned to 0 degrees
- moved J4 129.9 mm to (196.9, 121.9), turned to 180 degrees
- moved D4 129.7 mm to (180.3, 132.1), turned to -90 degrees
- moved R9 129.3 mm to (168.9, 128.3)
- moved U1 129.0 mm to (144.8, 61.3), turned to 180 degrees
- moved R6 125.2 mm to (182.9, 128.3)
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Routing:
- net +5V: track 0.00 -> 342.8 mm, vias 0 -> 1
- net /FAST_~{SLOW}: track 0.00 -> 97.9 mm, vias 0 -> 4
- net /FAST_CLK: track 0.00 -> 60.2 mm, vias 0 -> 4
- net /HLT: track 0.00 -> 55.3 mm, vias 0 -> 1
- net /LED_~{CLK}: track 0.00 -> 54.8 mm
- net /LED_CLK: track 0.00 -> 51.2 mm, vias 0 -> 3
- net /LED_PLS: track 0.00 -> 48.9 mm, vias 0 -> 2
- net /PULSE_CLK: track 0.00 -> 46.9 mm, vias 0 -> 4
- net /FAST_TR: track 0.00 -> 43.6 mm
- net /~{CLK}: track 0.00 -> 39.8 mm, vias 0 -> 2
- net /CLK: track 0.00 -> 39.5 mm, vias 0 -> 1
- net /PRE_CLK: track 0.00 -> 36.6 mm, vias 0 -> 6
- net /V_FUSE: track 0.00 -> 34.8 mm
- net /MODE_TR: track 0.00 -> 31.6 mm
- net /PLS_TR: track 0.00 -> 28.7 mm
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- added copper zone on F.Cu, net +5V
- added copper zone on F.Cu, net /VDD
- added copper zone on B.Cu, net GND
Other:
- board text added: "24 VDC Max"
- board text added: ">"
- board text added: "CLK"
- board text added: "FAST"
- board text added: "HLT"
- board text added: "JLCJLCJLCJLC"
- board text added: "MODE"
- board text added: "OFF"
- board text added: "ON"
- board text added: "PHI2"
- board text added: "PULSE"
- board text added: "Power Supply & 555 Clock"
- board text added: "RetroStack"
- board text added: "Rev 0"
- board text added: "~{CLK}"
- board text added: "©Microcode.io"
