File: boards/retro-stack-power-clock/retro-stack-power-clock.kicad_sch (KiCad schematic)
At the start: 54 parts, among them J1 BUS_6502, J2 DC_IN, J3 JMP_CLK_SEL, J4 JMP_HLT, SW1 SW_PWR, SW2 SW_MODE, SW3 SW_PULSE, U1 L7805CV, U2 74HC08, U3 74HC32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

Commit message: Rev 0 of the power and clock card ordered.
Parts:
- C2: Supplier Part 650-LVR125S-240 -> 581-TAP105K050SCS
- F1: Supplier Part 581-TAP105K050SCS -> 650-LVR125S-240
Changed lines of the file:
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@@
       (effects (font (size 1.27 1.27)) (justify left) hide)
     )
-    (property "Datasheet" "https://www.te.com/commerce/DocumentDelivery/DDEController?Action=showdoc&DocId=Catalog+Section%7FCLP00012%7FA%7Fpdf%7FEnglish%7FENG_CS_CLP00012_A_CLP00012.pdf%7FRF1251-000" (id 3) (at 62.23 29.21 0)
+    (property "Datasheet" "https://www.mouser.com/datasheet/2/40/tap-776819.pdf" (id 3) (at 62.23 29.21 0)
       (effects (font (size 1.27 1.27)) hide)
     )
@@
       (effects (font (size 1.27 1.27)) hide)
     )
-    (property "Supplier Part" "581-TAP105K050SCS " (id 6) (at 62.23 29.21 0)
+    (property "Supplier Part" "650-LVR125S-240" (id 6) (at 62.23 29.21 0)
       (effects (font (size 1.27 1.27)) hide)
     )
@@
       (effects (font (size 1.27 1.27)) hide)
     )
-    (property "Supplier Part" "650-LVR125S-240 " (id 6) (at 80.01 35.56 0)
-      (effects (font (size 1.27 1.27)) hide)
-    )
+    (property "Supplier Part" "581-TAP105K050SCS" (id 6) (at 80.01 35.56 0)
+      (effects (font (size 1.27 1.27)) hide)
+    )
