File: boards/retro-stack-cpu/retro-stack-cpu.kicad_pcb (KiCad board)
At the start: 2 copper layers, 99.1 x 99.1 mm, 29 parts, among them J1 BUS_6502, J2 TRM_PWR, SW1 SW_RESET, SW2 SW_CLK_EN, SW3 SW_RST_SEL, U2 DS1813, U3 W65C02SxP, X1 1Mhz

Commit message: Completed rev 0 of cpu, debug, and debug shield boards.
Other:
- board text added: "Rev 0"
Changed lines of the file:
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@@
     (attr board_only exclude_from_pos_files exclude_from_bom)
     (fp_text reference "kibuzzard-642C36EF" (at 0 -3.966104) (layer "F.SilkS") hide
-      (effects (font (size 0 0)))
+      (effects (font (size 0 0) (thickness 0.15)))
     )
     (fp_text value "G***" (at 0 3.966104) (layer "F.SilkS") hide
-      (effects (font (size 0 0)))
+      (effects (font (size 0 0) (thickness 0.15)))
     )
     (fp_poly (pts
@@
     (attr board_only exclude_from_pos_files exclude_from_bom)
     (fp_text reference "kibuzzard-642C367F" (at 0 -3.966104 90) (layer "F.SilkS") hide
-      (effects (font (size 0 0)))
+      (effects (font (size 0 0) (thickness 0.15)))
     )
     (fp_text value "G***" (at 0 3.966104 90) (layer "F.SilkS") hide
-      (effects (font (size 0 0)))
+      (effects (font (size 0 0) (thickness 0.15)))
     )
     (fp_poly (pts
@@
     (attr board_only exclude_from_pos_files exclude_from_bom)
     (fp_text reference "kibuzzard-642C33B0" (at 0 -3.974042 90) (layer "F.SilkS") hide
-      (effects (font (size 0 0)))
+      (effects (font (size 0 0) (thickness 0.15)))
     )
     (fp_text value "G***" (at 0 3.974042 90) (layer "F.SilkS") hide
-      (effects (font (size 0 0)))
+      (effects (font (size 0 0) (thickness 0.15)))
     )
     (fp_poly (pts
@@
     (attr board_only exclude_from_pos_files exclude_from_bom)
     (fp_text reference "kibuzzard-642C3375" (at 0 -3.974042 90) (layer "F.SilkS") hide
-      (effects (font (size 0 0)))
+      (effects (font (size 0 0) (thickness 0.15)))
     )
     (fp_text value "G***" (at 0 3.974042 90) (layer "F.SilkS") hide
-      (effects (font (size 0 0)))
+      (effects (font (size 0 0) (thickness 0.15)))
     )
     (fp_poly (pts
@@
       (effects (font (size 1.27 1.27) (thickness 0.254)))
     )
-    (fp_line (start -8.5 -0.254) (end -8.5 -2.5) (layer "F.SilkS") (width 0.2))
-    (fp_line (start 3.5 2.5) (end -6.985 2.5) (layer "F.SilkS") (width 0.2))
     (fp_line (start 3.5 -0.635) (end 3.5 2.5) (layer "F.SilkS") (width 0.2))
-    (fp_line (start 0 2.9) (end 0 2.9) (layer "F.SilkS") (width 0.1))
     (fp_line (start -8.5 -2.5) (end 1.524 -2.5) (layer "F.SilkS") (width 0.2))
+    (fp_line (start 0 2.9) (end 0 2.9) (layer "F.SilkS") (width 0.1))
+    (fp_line (start 3.5 2.5) (end -6.985 2.5) (layer "F.SilkS") (width 0.2))
+    (fp_line (start -8.5 -0.254) (end -8.5 -2.5) (layer "F.SilkS") (width 0.2))
     (fp_line (start 0 3) (end 0 3) (layer "F.SilkS") (width 0.1))
     (fp_arc (start 0 2.9) (mid 0.05 2.95) (end 0 3) (layer "F.SilkS") (width 0.1))
     (fp_arc (start 0 3) (mid -0.05 2.95) (end 0 2.9) (layer "F.SilkS") (width 0.1))
-    (fp_line (start -10.1 -4.1) (end 16.7 -4.1) (layer "F.CrtYd") (width 0.1))
+    (fp_line (start -10.1 3.5) (end -10.1 -4.1) (layer "F.CrtYd") (width 0.1))
     (fp_line (start 16.7 -4.1) (end 16.7 3.5) (layer "F.CrtYd") (width 0.1))
+    (fp_line (start -10.1 -4.1) (end 16.7 -4.1) (layer "F.CrtYd") (width 0.1))
     (fp_line (start 16.7 3.5) (end -10.1 3.5) (layer "F.CrtYd") (width 0.1))
-    (fp_line (start -10.1 3.5) (end -10.1 -4.1) (layer "F.CrtYd") (width 0.1))
-    (fp_line (start -8.5 -2.5) (end 3.5 -2.5) (layer "F.Fab") (width 0.1))
-    (fp_line (start 9.6 -2.5) (end 15.7 -2.5) (layer "F.Fab") (width 0.1))
-    (fp_line (start 3.5 -1.25) (end 9.6 -1.25) (layer "F.Fab") (width 0.1))
-    (fp_line (start 3.5 2.5) (end -8.5 2.5) (layer "F.Fab") (width 0.1))
-    (fp_line (start 15.7 -2.5) (end 15.7 2.5) (layer "F.Fab") (width 0.1))
-    (fp_line (start 3.5 -2.5) (end 3.5 2.5) (layer "F.Fab") (width 0.1))
     (fp_line (start -8.5 2.5) (end -8.5 -2.5) (layer "F.Fab") (width 0.1))
+    (fp_line (start 9.6 -2.5) (end 15.7 -2.5) (layer "F.Fab") (width 0.1))
+    (fp_line (start -8.5 -2.5) (end 3.5 -2.5) (layer "F.Fab") (width 0.1))
+    (fp_line (start 9.6 -1.25) (end 9.6 -2.5) (layer "F.Fab") (width 0.1))
     (fp_line (start 9.6 1.2) (end 3.5 1.2) (layer "F.Fab") (width 0.1))
     (fp_line (start 15.7 2.5) (end 9.6 2.5) (layer "F.Fab") (width 0.1))
+    (fp_line (start 3.5 -1.25) (end 9.6 -1.25) (layer "F.Fab") (width 0.1))
+    (fp_line (start 15.7 -2.5) (end 15.7 2.5) (layer "F.Fab") (width 0.1))
     (fp_line (start 9.6 -1.25) (end 9.6 1.2) (layer "F.Fab") (width 0.1))
+    (fp_line (start 3.5 2.5) (end -8.5 2.5) (layer "F.Fab") (width 0.1))
     (fp_line (start 9.6 2.5) (end 9.6 1.25) (layer "F.Fab") (width 0.1))
-    (fp_line (start 9.6 -1.25) (end 9.6 -2.5) (layer "F.Fab") (width 0.1))
+    (fp_line (start 3.5 -2.5) (end 3.5 2.5) (layer "F.Fab") (width 0.1))
     (pad "1" thru_hole rect (at 0 0 270) (size 1.4 1.4) (drill 0.9) (layers *.Cu *.Mask)
       (net 1 "GND") (pinfunction "A") (pintype "passive"))
@@
     (attr board_only exclude_from_pos_files exclude_from_bom)
     (fp_text reference "kibuzzard-642C3403" (at 0 -3.974042 90) (layer "F.SilkS") hide
-      (effects (font (size 0 0)))
+      (effects (font (size 0 0) (thickness 0.15)))
     )
     (fp_text value "G***" (at 0 3.974042 90) (layer "F.SilkS") hide
-      (effects (font (size 0 0)))
+      (effects (font (size 0 0) (thickness 0.15)))
     )
     (fp_poly (pts
@@
     (effects (font (size 1 1) (thickness 0.153)) (justify left))
   )
+  (gr_text "Rev 0" (at 106.68 127.762) (layer "F.SilkS")
+    (effects (font (size 1 1) (thickness 0.153)))
+  )
   (gr_text "JLCJLCJLCJLC" (at 167.64 102.235 90) (layer "F.SilkS")
