File: boards/retro-stack-cpu/retro-stack-cpu.kicad_sch (KiCad schematic)
At the start: 22 parts, among them J1 BUS_6502, J2 TRM_PWR, SW1 SW_RESET, SW2 SW_CLK_EN, SW3 SW_RST_SEL, U2 DS1813, U3 W65C02SxP, X1 1Mhz

Commit message: Completed rev 0 of cpu, debug, and debug shield boards.
Parts:
- R5: Mfr (none) -> Vishay; Mfr Part (none) -> MBA02040C1001FCT00; Supplier (none) -> Mouser; Supplier Part (none) -> 594-MBA02040C1001FCT
- R6: Mfr (none) -> Vishay; Mfr Part (none) -> MBA02040C3309FC100; Supplier (none) -> Mouser; Supplier Part (none) -> 594-5063JD33R00F1
Changed lines of the file:
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@@
       (effects (font (size 1.27 1.27)) hide)
     )
-    (property "Datasheet" "~" (id 3) (at 100.33 52.07 0)
+    (property "Datasheet" "https://www.mouser.com/datasheet/2/427/mbxsma-1286643.pdf" (id 3) (at 100.33 52.07 0)
+      (effects (font (size 1.27 1.27)) hide)
+    )
+    (property "Mfr" "Vishay" (id 4) (at 100.33 52.07 0)
+      (effects (font (size 1.27 1.27)) hide)
+    )
+    (property "Mfr Part" "MBA02040C3309FC100 " (id 5) (at 100.33 52.07 0)
+      (effects (font (size 1.27 1.27)) hide)
+    )
+    (property "Supplier Part" "594-5063JD33R00F1 " (id 6) (at 100.33 52.07 0)
+      (effects (font (size 1.27 1.27)) hide)
+    )
+    (property "Supplier" "Mouser" (id 7) (at 100.33 52.07 0)
       (effects (font (size 1.27 1.27)) hide)
     )
@@
       (effects (font (size 1.27 1.27)) hide)
     )
-    (property "Datasheet" "~" (id 3) (at 189.23 60.96 0)
+    (property "Datasheet" "https://www.mouser.com/datasheet/2/427/mbxsma-1286643.pdf" (id 3) (at 189.23 60.96 0)
       (effects (font (size 1.27 1.27)) hide)
     )
+    (property "Mfr" "Vishay" (id 4) (at 189.23 60.96 0)
+      (effects (font (size 1.27 1.27)) hide)
+    )
+    (property "Mfr Part" "MBA02040C1001FCT00 " (id 5) (at 189.23 60.96 0)
+      (effects (font (size 1.27 1.27)) hide)
+    )
+    (property "Supplier Part" "594-MBA02040C1001FCT" (id 6) (at 189.23 60.96 0)
+      (effects (font (size 1.27 1.27)) hide)
+    )
+    (property "Supplier" "Mouser" (id 7) (at 189.23 60.96 0)
+      (effects (font (size 1.27 1.27)) hide)
+    )
