File: boards/retro-stack-debug/retro-stack-debug.kicad_sch (KiCad schematic)
At the start: 39 parts, among them J1 BUS_6502, J2 TRM_PWR, J3 BUS_DEBUG, SW1 SW_ENABLE, U1 74HC244, U2 74HC244, U3 74HC244, U4 74HC240

Commit message: Update documentation for recently completed board revisions.
Other:
- note added: "Address & Data Buffers"
- note added: "Control Signal Buffer"
- note added: "Signal LEDs"
- note added: "Signals Enable"
- moved on the sheet: R2, SW1
