File: boards/retro-stack-template/retro-stack-template.kicad_sch (KiCad schematic)
At the start: 5 parts, among them J1 BUS_6502

Commit message: Update template
Parts:
- added D1: LED_PWR, LED_THT:LED_D5.0mm, symbol Device:LED
- added J2: TRM_PWR, TerminalBlock_Phoenix:TerminalBlock_Phoenix_MPT-0,5-2-2.54_1x02_P2.54mm_Horizontal, symbol Connector:Screw_Terminal_01x02
- added R1: 1k, Resistor_THT:R_Axial_DIN0204_L3.6mm_D1.6mm_P5.08mm_Horizontal, symbol Device:R
Connections:
- net VSS is gone; now on net GND: J1.39 (Pin_39)
- net GND: now also J2.2 (Pin_2), R1.2
- net VDD renamed +5V
- net +5V: now also D1.2 (A), J2.1 (Pin_1)
- new net: D1.1 (K), R1.1
Other:
- note added: "External Power"
- note added: "Power LED"

Commit message: Update template to use right angle idc instead of vertical pin socket.
Parts:
- J1: footprint Connector_PinSocket_2.54mm:PinSocket_2x20_P2.54mm_Vertical -> Connector_IDC:IDC-Header_2x20_P2.54mm_Horizontal
Connections:
- net +5V: now also J1.15 (Pin_15); no longer J1.16 (Pin_16)
- net A0: now also J1.17 (Pin_17); no longer J1.18 (Pin_18)
- net A1: now also J1.19 (Pin_19); no longer J1.20 (Pin_20)
- net A10: now also J1.37 (Pin_37); no longer J1.38 (Pin_38)
- net A11: now also J1.39 (Pin_39); no longer J1.40 (Pin_40)
- net A12: now also J1.38 (Pin_38); no longer J1.37 (Pin_37)
- net A13: now also J1.36 (Pin_36); no longer J1.35 (Pin_35)
- net A14: now also J1.34 (Pin_34); no longer J1.33 (Pin_33)
- net A15: now also J1.32 (Pin_32); no longer J1.31 (Pin_31)
- net A2: now also J1.21 (Pin_21); no longer J1.22 (Pin_22)
- net A3: now also J1.23 (Pin_23); no longer J1.24 (Pin_24)
- net A4: now also J1.25 (Pin_25); no longer J1.26 (Pin_26)
- net A5: now also J1.27 (Pin_27); no longer J1.28 (Pin_28)
- net A6: now also J1.29 (Pin_29); no longer J1.30 (Pin_30)
- net A7: now also J1.31 (Pin_31); no longer J1.32 (Pin_32)
- net A8: now also J1.33 (Pin_33); no longer J1.34 (Pin_34)
- net A9: now also J1.35 (Pin_35); no longer J1.36 (Pin_36)
- net BE: now also J1.10 (Pin_10); no longer J1.9 (Pin_9)
- net D0: now also J1.16 (Pin_16); no longer J1.15 (Pin_15)
- net D1: now also J1.18 (Pin_18); no longer J1.17 (Pin_17)
- net D2: now also J1.20 (Pin_20); no longer J1.19 (Pin_19)
- net D3: now also J1.22 (Pin_22); no longer J1.21 (Pin_21)
- net D4: now also J1.24 (Pin_24); no longer J1.23 (Pin_23)
- net D5: now also J1.26 (Pin_26); no longer J1.25 (Pin_25)
- net D6: now also J1.28 (Pin_28); no longer J1.27 (Pin_27)
- net D7: now also J1.30 (Pin_30); no longer J1.29 (Pin_29)
- net GND: now also J1.40 (Pin_40); no longer J1.39 (Pin_39)
- net NC: now also J1.12 (Pin_12); no longer J1.11 (Pin_11)
- net PHI1O: now also J1.5 (Pin_5); no longer J1.6 (Pin_6)
- net PHI2: now also J1.8 (Pin_8); no longer J1.7 (Pin_7)
- net PHI2O: now also J1.4 (Pin_4); no longer J1.3 (Pin_3)
- net RDY: now also J1.3 (Pin_3); no longer J1.4 (Pin_4)
- net R/~{W}: now also J1.14 (Pin_14); no longer J1.13 (Pin_13)
- net SYNC: now also J1.13 (Pin_13); no longer J1.14 (Pin_14)
- net VPB: now also J1.1 (Pin_1); no longer J1.2 (Pin_2)
- net ~{IRQ}: now also J1.7 (Pin_7); no longer J1.8 (Pin_8)
- net ~{ML}: now also J1.9 (Pin_9); no longer J1.10 (Pin_10)
- net ~{NMI}: now also J1.11 (Pin_11); no longer J1.12 (Pin_12)
- net ~{RES}: now also J1.2 (Pin_2); no longer J1.1 (Pin_1)
- net ~{SO}: now also J1.6 (Pin_6); no longer J1.5 (Pin_5)
