File: boards/pld-test/pld-test.kicad_sch (KiCad schematic)
At the start: 6 parts, among them U1 ATF16V8B-15PU, U2 74LS151

Commit message: First working memory pld coded.
Parts:
- removed C3: 0u1, symbol Device:C_Small
- removed U2: 74LS151, symbol 74xx:74LS151
- added BAR?: HDSP-4830_2, Display:HDSP-4830, symbol LED:HDSP-4830_2
- added RN?: 1k, Resistor_THT:R_Array_SIP9, symbol Device:R_Network08
Connections:
- net ~{OUT}4 is gone; now on net ~{ROM_OE}: U1.15 (I/O4)
- net ~{OUT}5 is gone; now on net ~{ROM_CS}: U1.16 (I/O5)
- net ~{OUT}6 is gone; now on net ~{RAM_WE}: U1.17 (I/O6)
- net ~{OUT}7 is gone; now on net ~{RAM_OE}: U1.18 (I/O7)
- net ~{OUT}8 is gone; now on net ~{RAM_CS}: U1.19 (I/O8)
- net GND: now also RN?.1 (common)
- net ~{ROM_OE}: now reaches A1.23 (SDA/A4)
- net ~{ROM_OE}: now also BAR?.5 (A)
- net RESULT renamed ~{RAM_CS}
- net ~{RAM_CS}: now also BAR?.1 (A)
- net RS0 renamed ~{RAM_OE}
- net ~{RAM_OE}: now also BAR?.2 (A)
- net RS1 renamed ~{RAM_WE}
- net ~{RAM_WE}: now also BAR?.3 (A)
- net RS2 renamed ~{ROM_CS}
- net ~{ROM_CS}: now also BAR?.4 (A)
- net ~{OE}: no longer names the net of A1.25 (A6)
- net ~{OE}: no longer U1.11 (I9/~{OE})
- net ~{OUT}1: no longer names the net of U1.12 (I/O1)
- net ~{OUT}2: no longer names the net of U1.13 (I/O2)
- net ~{OUT}3: no longer names the net of U1.14 (I/O3)
- new net: BAR?.20 (K), RN?.2 (R1)
- new net: BAR?.19 (K), RN?.3 (R2)
- new net: BAR?.18 (K), RN?.4 (R3)
- new net: BAR?.17 (K), RN?.5 (R4)
- new net: BAR?.16 (K), RN?.6 (R5)
- new net: BAR?.15 (K), RN?.7 (R6)
- new net: BAR?.14 (K), RN?.8 (R7)
- new net: BAR?.13 (K), RN?.9 (R8)
- no-connect marks 12 -> 22

Commit message: Initial PLD test and RAM/ROM board.
Parts:
- removed BAR?: HDSP-4830_2, Display:HDSP-4830, symbol LED:HDSP-4830_2
- removed C1: 10u, symbol Device:C_Polarized
- removed RN?: 1k, Resistor_THT:R_Array_SIP9, symbol Device:R_Network08
- added C1: 10u, Capacitor_THT:CP_Radial_D5.0mm_P2.50mm, symbol Device:C_Polarized_Small
- added C10, C3, C4, C5, C6, C8: 1u, Capacitor_THT:C_Rect_L4.0mm_W2.5mm_P2.50mm, symbol Device:C_Small
- added C11, C7, C9: 0u1, Capacitor_THT:C_Rect_L4.0mm_W2.5mm_P2.50mm, symbol Device:C_Small
- added J1: HDR_TM1620DSP, Connector_PinHeader_2.54mm:PinHeader_2x05_P2.54mm_Vertical, symbol Connector_Generic:Conn_02x05_Odd_Even
- added J2: HDR_SD, Connector_PinHeader_2.54mm:PinHeader_1x07_P2.54mm_Vertical, symbol Connector_Generic:Conn_01x07
- added J3: HDR_IN, Connector_PinSocket_2.54mm:PinSocket_1x09_P2.54mm_Vertical, symbol Connector:Conn_01x09_Female
- added J4: HDR_OUT, Connector_PinSocket_2.54mm:PinSocket_1x09_P2.54mm_Vertical, symbol Connector:Conn_01x09_Female
- added R1, R2, R3, R4, R5, R6, R7, R8, R9: 1k, Resistor_THT:R_Axial_DIN0204_L3.6mm_D1.6mm_P5.08mm_Horizontal, symbol Device:R_Small
- added SW1: SW_Left, Button_Switch_THT:SW_PUSH_6mm, symbol Switch:SW_Push
- added SW2: SW_Right, Button_Switch_THT:SW_PUSH_6mm, symbol Switch:SW_Push
- added SW3: SW_Menu, Button_Switch_THT:SW_PUSH_6mm, symbol Switch:SW_Push
- added SW4: SW_Select, Button_Switch_THT:SW_PUSH_6mm, symbol Switch:SW_Push
- added SW5: SW_RST, Button_Switch_THT:SW_PUSH_6mm, symbol Switch:SW_Push
- added U2: 74HC14, Package_DIP:DIP-14_W7.62mm_Socket_LongPads, symbol 74xx:74HC14
- added U3: MCP23S17_SP, Package_DIP:DIP-28_W7.62mm_Socket_LongPads, symbol Interface_Expansion:MCP23S17_SP
- A1: Man Part # (none) -> ABX00028; Manufacturer (none) -> Arduino; Supp Part # (none) -> 782-ABX00028; Supplier (none) -> Mouser
- C2: value 0u1 -> 1u; footprint (none) -> Capacitor_THT:C_Rect_L4.0mm_W2.5mm_P2.50mm; Man Part # (none) -> FA18X7R1E105KRU06; Manufacturer (none) -> TDK; Supp Part # (none) -> 810-FA18X7R1E105KRU6; Supplier (none) -> Mouser
- U1: Man Part # (none) -> ATF16V8B-15PU; Manufacturer (none) -> Microchip; Supp Part # (none) -> 556-AF16V8B15PU; Supplier (none) -> Mouser
Connections:
- net +5V: now also C1.1, C10.1, C11.1, C6.1, C7.1, C8.1, C9.1, J1.1 (Pin_1), J1.2 (Pin_2), J2.7 (Pin_7), R1.2, R3.2, R5.2, R7.2, R9.2, U2.14 (VCC), U3.9 (VDD); no longer A1.28 (~{RESET}), A1.3 (~{RESET}), C2.1
- net CLK: now also J3.1 (Pin_1)
- net GND: now also C1.2, C10.2, C11.2, C3.2, C4.2, C5.2, C6.2, C7.2, C8.2, C9.2, J1.10 (Pin_10), J1.9 (Pin_9), J2.1 (Pin_1), SW1.1, SW2.1, SW3.1, SW4.1, SW5.2, U2.11, U2.13, U2.7 (GND), U3.10 (VSS), U3.15 (A0), U3.16 (A1), U3.17 (A2)
- net MOSI: now reaches A1.14 (MOSI)
- net MOSI: now also J2.5 (Pin_5), U3.13 (SI)
- net MISO: now reaches A1.15 (MISO)
- net MISO: now also J2.3 (Pin_3), U3.14 (SO)
- net SCK: now reaches A1.16 (SCK)
- net SCK: now also J2.4 (Pin_4), U3.12 (SCK)
- net In9/~{OE}: now reaches U1.11 (I9/~{OE})
- net In9/~{OE}: now also A1.7 (D4), J4.9 (Pin_9)
- net Out1: now reaches U1.12 (I/O1)
- net Out1: now also J4.8 (Pin_8), U3.21 (GPA0)
- net Out2: now reaches U1.13 (I/O2)
- net Out2: now also J4.7 (Pin_7), U3.22 (GPA1)
- net Out3: now reaches U1.14 (I/O3)
- net Out3: now also J4.6 (Pin_6), U3.23 (GPA2)
- net A10 renamed DSP_STB
- net DSP_STB: now also J1.3 (Pin_3), J1.4 (Pin_4); no longer U1.4 (I3)
- net A11 renamed DSP_CLK
- net DSP_CLK: now also J1.5 (Pin_5), J1.6 (Pin_6); no longer U1.5 (I4)
- net A12 renamed DSP_DIN
- net DSP_DIN: now also J1.7 (Pin_7), J1.8 (Pin_8); no longer U1.6 (I5)
- net A13 renamed In6
- net In6: now also J3.7 (Pin_7), U3.6 (GPB5); no longer A1.11 (D8)
- net A14 renamed In7
- net In7: now also J3.8 (Pin_8), U3.7 (GPB6); no longer A1.12 (D9)
- net A15 renamed GPIO_~{CS}
- net GPIO_~{CS}: now also U3.11 (~{CS}); no longer U1.9 (I8)
- net A9 renamed In2
- net In2: now also J3.3 (Pin_3), U3.2 (GPB1); no longer A1.7 (D4)
- net R/~{W} renamed GPIO_~{RST}
- net GPIO_~{RST}: now also U3.18 (~{RESET}); no longer U1.2 (I1)
- net ~{RAM_CS} renamed BTN_LEFT
- net BTN_LEFT: now also U2.2; no longer U1.19 (I/O8)
- net ~{RAM_OE} renamed BTN_RIGHT
- net BTN_RIGHT: now also U2.4; no longer U1.18 (I/O7)
- net ~{RAM_WE} renamed BTN_MENU
- net BTN_MENU: now also U2.6; no longer U1.17 (I/O6)
- net ~{ROM_CS} renamed BTN_SEL
- net BTN_SEL: now also U2.8; no longer U1.16 (I/O5)
- net ~{ROM_OE}: no longer names the net of A1.23 (SDA/A4)
- net ~{ROM_OE}: no longer U1.15 (I/O4)
- new net In1: J3.2 (Pin_2), U1.2 (I1), U3.1 (GPB0)
- new net In3: J3.4 (Pin_4), U1.4 (I3), U3.3 (GPB2)
- new net In4: J3.5 (Pin_5), U1.5 (I4), U3.4 (GPB3)
- new net In5: J3.6 (Pin_6), U1.6 (I5), U3.5 (GPB4)
- new net In8: J3.9 (Pin_9), U1.9 (I8), U3.8 (GPB7)
- new net Out4: J4.5 (Pin_5), U1.15 (I/O4), U3.24 (GPA3)
- new net Out5: J4.4 (Pin_4), U1.16 (I/O5), U3.25 (GPA4)
- new net Out6: J4.3 (Pin_3), U1.17 (I/O6), U3.26 (GPA5)
- new net Out7: J4.2 (Pin_2), U1.18 (I/O7), U3.27 (GPA6)
- new net Out8: J4.1 (Pin_1), U1.19 (I/O8), U3.28 (GPA7)
- new net RC_LEFT: C2.1, R2.2, U2.1
- new net RC_MENU: C4.1, R6.2, U2.5
- new net RC_RIGHT: C3.1, R4.2, U2.3
- new net RC_SEL: C5.1, R8.2, U2.9
- new net SD_CD: A1.11 (D8), J2.2 (Pin_2)
- new net SD_~{CS}: A1.12 (D9), J2.6 (Pin_6)
- new net VD_L: R1.1, R2.1, SW1.2
- new net VD_M: R5.1, R6.1, SW3.2
- new net VD_R: R3.1, R4.1, SW2.2
- new net VD_S: R7.1, R8.1, SW4.2
- new net ~{RESET}: A1.28 (~{RESET}), A1.3 (~{RESET}), R9.1, SW5.1
- no-connect marks 22 -> 13
Other:
- note added: "Arduino Socket & Reset"
- note added: "Buttons & HW Debounce"
- note added: "MicroSD & Display Modules"
- note added: "PLD Socket & SPI GPIO Expander"
- company: (none) -> Microcode.io
- title: (none) -> RetroStack - PLD Tester
- moved on the sheet: A1, U1
