File: boards/retro-stack-ram-rom/retro-stack-ram-rom.kicad_sch (KiCad schematic)
At the start: 25 parts, among them J1 BUS_6502, J2 TRM_PWR, U1 74HC14, U2 28C256, U3 AS6C62256, U4 ATF16V8B-15PU

Commit message: Initial PLD test and RAM/ROM board.
Parts:
- removed R1: 1k, Resistor_THT:R_Axial_DIN0204_L3.6mm_D1.6mm_P5.08mm_Horizontal, symbol Device:R
- U2: footprint Package_DIP:DIP-28_W15.24mm_Socket_LongPads -> RetroStack:28655410
Connections:
- net at D2.1 (K): now also RN1.3 (R2); no longer RN1.2 (R1)
- net PWR_R: now reaches D1.1 (K)
- net PWR_R: now also RN1.2 (R1)
- net at D5.1 (K): now also RN1.6 (R5); no longer RN1.5 (R4)
- net at D4.1 (K): now also RN1.5 (R4); no longer RN1.4 (R3)
- net at D3.1 (K): now also RN1.4 (R3); no longer RN1.3 (R2)
- net at D6.1 (K): now also RN1.7 (R6); no longer RN1.6 (R5)
- no-connect marks 8 -> 7
Other:
- note added: "*ZIF Socket Aries 28-6554-10"
